File: SpeccyPower5v.brd (EAGLE design)
At the start: 112.4 x 40 mm, 67 parts, among them T1 TRANS_ER29

Commit message: .
Parts:
- removed 1RZ1: (no value), varistor:S1210
- removed 2R1: 220k 1w, rcl:P0613/15
- removed 2R1A1, 2R1C1, 2R1E1: 120k, rcl:M0805
- removed 2R1B1, 2R1D1, 2R1F1: 150k, rcl:M0805
- removed 3R1, 3R2: 0, rcl:M1206
- added 3R8: (no value), rcl:R0805
- added S1, S2: (no value), pinhead:1X01
- 3VD2: value MA10799 -> (none); device diode:TO220ABS -> diode:DO220S
- moved 2R1A 2.56 mm to (87.6, 90.5), turned to 180 degrees
- moved 3VD2 1.80 mm to (141.0, 61.9)
- moved 1TH1 1.62 mm to (67.0, 87.3), turned to 270 degrees
- moved 2R1B 1.14 mm to (86.7, 87.3)
- moved SV2 0.64 mm to (149.5, 87.0)
- moved 3R6 0.64 mm to (145.1, 82.5)
- moved 3R7 0.64 mm to (140.3, 82.5)
- moved SV1 0.63 mm to (41.3, 80.3)
- moved 3L2 0.63 mm to (149.9, 79.4)
- moved 2R4 0.45 mm to (110.5, 74.9)
- moved 3C3 0.32 mm to (141.6, 78.7)
- moved 1L1 0.32 mm to (70.2, 71.8)
- moved 1C2 0.32 mm to (59.4, 75.6)
- moved 2C11 0.32 mm to (124.1, 85.7)
- moved 3C2 0.32 mm to (134.9, 72.1)
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Connections:
- removed net N$27: 2R1C1.1, 2R1D1.1, 2R1E1.2, 2R1F1.1
- removed net N$31: 2R1A1.1, 2R1B1.1, 2R1C1.2, 2R1D1.2
- removed net N$33: 2C11.1, 3R2.1
- new net N$36: S2.1, SV1.1
- net +5V: now also 3R8.2
- net -IN: now also 2C11.1; no longer 3R2.2
- net N$26: now also 3R8.1
- net N$28: now also 3VD2.A; no longer 3VD2.A1, 3VD2.A2
- net N$32: now also S1.1; no longer SV1.1
Routing:
- net -IN: track 71.7 -> 87.8 mm
- net N$28: track 20.5 -> 7.67 mm
- net N$33: track 13.3 -> 3.49 mm
- net N$31: track 13.9 -> 4.13 mm
- net N$32: track 17.4 -> 9.43 mm
- net N$37: track 0.00 -> 6.10 mm
- net N$36: track 0.00 -> 5.74 mm
- net N$34: track 0.00 -> 5.08 mm
- net N$27: track 0.00 -> 3.81 mm
- net N$2: track 11.6 -> 14.6 mm
- net N$26: track 2.41 -> 4.95 mm
- net N$13: track 73.7 -> 75.0 mm
- net N$44: track 8.54 -> 7.47 mm
- net N$45: track 9.99 -> 9.14 mm
- net N$23: track 68.5 -> 69.4 mm
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Other:
- board size 112.4 x 40 mm -> 112.1 x 40 mm

Commit message: test v h
Parts:
- added 2C4A, 2C5A, 2C7A: (no value), rcl:C0805
- moved 2R1E 41.4 mm to (54.3, 68.6)
- moved 2R1F 41.4 mm to (54.3, 70.8)
- moved 2R3 41.3 mm to (70.2, 39.4)
- moved 2R1C 40.9 mm to (47.3, 69.5)
- moved 2R1D 40.9 mm to (49.8, 69.5)
- moved 2DA1 40.5 mm to (101.6, 63.2)
- moved 1DA1 40.5 mm to (75.6, 63.2)
- moved 1PC1 40.5 mm to (94.6, 68.6)
- moved 2C6 40.5 mm to (72.7, 61.9)
- moved 2R16 40.5 mm to (100.6, 59.1)
- moved 2R5 40.5 mm to (80.6, 69.5)
- moved 2R8 40.5 mm to (72.7, 64.5)
- moved 2VD1 40.5 mm to (81.3, 52.4)
- moved 2C10 40.5 mm to (104.8, 56.5)
- moved 2C5 40.5 mm to (69.2, 61.9)
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Connections:
- net N$23 renamed +IN
- removed net N$40: 1DA1.2, 1PC1.3, 2C4.2, 2R5.1, 2R7.2
- removed net N$6: 1DA1.1, 2C4.1, 2R5.2
- new net 817-3: 1DA1.2, 1PC1.3, 2C4.2, 2C4A.2, 2R5.1, 2R7.2
- new net COMP: 1DA1.1, 2C4.1, 2C4A.1, 2R5.2
- net -IN: now also 2C5A.2, 2C7A.2
- net N$3: now also 2C5A.1
- net N$4: now also 2C7A.1
Routing:
- net 817-3: track 0.00 -> 28.8 mm
- net N$40: track 27.6 -> 0.00 mm
- net COMP: track 0.00 -> 13.1 mm
- net N$6: track 12.2 -> 0.00 mm
- net +16IN: track 67.8 -> 61.7 mm
- net -IN: track 87.8 -> 92.0 mm
- net N$33: track 3.49 -> 5.40 mm
- net N$3: track 5.08 -> 6.67 mm
- net N$29: track 14.8 -> 13.6 mm
- net N$30: track 10.9 -> 10.1 mm
- net N$19: track 9.03 -> 8.28 mm
- net N$31: track 4.13 -> 4.76 mm
- net N$1: track 11.2 -> 10.6 mm
- net N$8: track 8.99 -> 8.35 mm
- net N$27: track 3.81 -> 4.45 mm
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Other:
- board size 112.1 x 40 mm -> 112.1 x 38.1 mm

Commit message: ..
Parts:
- 2R13: device rcl:0207/10 -> rcl:0204/7
- 2VD2: device SpeccyPower5v:DO35-10 -> SpeccyPower5v:DO35-7
- 3L2: device rcl:TFI0305 -> rcl:LAL02
- 3R7: device rcl:M1206 -> rcl:M0805
- moved 3L2 16.8 mm to (113.0, 68.9), turned to 270 degrees
- moved 2C10 8.26 mm to (105.1, 64.8)
- moved 3C3 7.68 mm to (104.5, 56.5), flipped to the bottom, turned to 90 degrees
- moved SV2 6.68 mm to (113.0, 63.8), turned to 0 degrees
- moved 2R14 6.07 mm to (102.9, 65.4), turned to 90 degrees
- moved 3R8 4.69 mm to (110.5, 56.8), turned to 270 degrees
- moved 3R7 3.51 mm to (109.5, 60.0)
- moved 2R13 2.71 mm to (107.3, 67.6)
- moved 3R6 1.93 mm to (112.7, 56.8), turned to 270 degrees
- moved 2VD2 1.42 mm to (62.9, 49.8)
- moved 2R12 1.27 mm to (102.9, 70.2)
- moved 2DA1 0.95 mm to (100.6, 63.2)
- moved 1VD2 0.64 mm to (48.6, 42.5)
- moved 1VD4 0.64 mm to (52.1, 42.5)
- moved 2R3 0.64 mm to (70.2, 40.0), turned to 355 degrees
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Routing:
- net +16IN: track 61.7 -> 25.8 mm
- net +5V: track 14.3 -> 23.8 mm
- net GND: track 68.8 -> 62.5 mm
- net N$42: track 14.2 -> 12.0 mm
- net N$12: track 7.14 -> 9.08 mm
- net N$13: track 74.4 -> 72.7 mm
- net -IN: track 92.0 -> 90.4 mm
- net +IN: track 68.9 -> 68.0 mm
- net N$33: track 5.40 -> 4.76 mm
- net N$31: track 4.76 -> 4.13 mm
- net N$14: track 7.53 -> 6.93 mm
- net N$26: track 4.95 -> 4.45 mm
Other:
- board size 112.1 x 38.1 mm -> 112.1 x 37.5 mm

Commit message: ..
Parts:
- moved 1VD3 2.56 mm to (54.3, 55.6), turned to 325 degrees
- moved 1VD4 2.03 mm to (53.3, 44.1)
- moved 1VD1 1.42 mm to (49.2, 53.0), turned to 100 degrees
- moved 2R3 0.71 mm to (69.5, 40.3), turned to 350 degrees
- moved 1C7 0.63 mm to (60.3, 66.0)
- moved 1F1 0.32 mm to (26.0, 68.9)
- moved 1L1 0.32 mm to (39.7, 46.7)
- moved 2C2 0.32 mm to (58.1, 42.5)
- moved 1TH1 0.32 mm to (36.5, 61.6)
- moved 1VD2 0.32 mm to (48.6, 42.9)
- moved 2R13 0.32 mm to (107.3, 67.3)
- moved 2R5 0.32 mm to (80.6, 69.2)
- moved 2R7 0.32 mm to (72.1, 71.1)
- moved 3L2 0.32 mm to (113.0, 68.6)
Routing:
- net N$1: track 10.6 -> 8.47 mm
- net -IN: track 90.4 -> 88.4 mm
- net +IN: track 68.0 -> 66.0 mm
- net N$44: track 7.69 -> 9.19 mm
- net N$30: track 9.72 -> 8.65 mm
- net N$45: track 9.14 -> 8.51 mm
Other:
- board size 112.1 x 37.5 mm -> 112.1 x 36.8 mm

Commit message: ..
Parts:
- removed 3R8: (no value), rcl:R0805
- 3C3: device SpeccyPower5v:TT2D7L -> SpeccyPower5v:TT2D7L-2
- 3R7: value 0 -> (none); device rcl:M0805 -> rcl:R0805
- moved 2R13 4.76 mm to (102.6, 67.3)
- moved 3R7 3.38 mm to (107.3, 57.5), turned to 90 degrees
- moved 3R6 3.24 mm to (109.5, 57.5), turned to 90 degrees
- moved 2R14 2.93 mm to (105.7, 64.8), turned to 180 degrees
- moved 2R12 2.58 mm to (105.4, 70.6)
- moved 3L2 2.42 mm to (110.8, 69.5), turned to 225 degrees
- moved SV2 1.27 mm to (114.3, 63.8)
- moved 2DA1 0.63 mm to (100.0, 63.2)
- flipped 3C3 to the top, turned to 270 degrees
Connections:
- removed net N$42: 2C10.1, 2DA1.R, 2R16.2, 3R7.1
- net +5V: now also 3R7.2; no longer 3R8.2
- net N$26: now also 2C10.1, 2DA1.R, 2R16.2, 3R7.1; no longer 3R7.2, 3R8.1
Routing:
- net N$26: track 4.45 -> 17.2 mm
- net N$42: track 12.0 -> 0.00 mm
- net GND: track 62.5 -> 52.5 mm
- net +5V: track 23.5 -> 26.2 mm
- net N$12: track 9.07 -> 7.27 mm
- net N$14: track 7.18 -> 5.46 mm
- net N$16: track 2.42 -> 3.49 mm

Commit message: ..
Parts:
- 2R9: device rcl:0207/10 -> rcl:0204/7
- 2VD2: device SpeccyPower5v:DO35-7 -> SpeccyPower5v:DO35-10
- moved 3L2 26.6 mm to (104.1, 43.8)
- moved 1C7 26.3 mm to (53.7, 40.6)
- moved 1DA1 26.3 mm to (68.9, 37.8)
- moved 1TH1 26.3 mm to (29.8, 36.2)
- moved 1VD2 26.3 mm to (41.9, 17.5)
- moved 1VD4 26.3 mm to (46.7, 18.7)
- moved 2C10 26.3 mm to (98.4, 39.4)
- moved 2C4 26.3 mm to (77.8, 40.0)
- moved 2C4A 26.3 mm to (77.8, 40.0)
- moved 2C5 26.3 mm to (62.5, 36.5)
- moved 2C5A 26.3 mm to (62.5, 36.5)
- moved 2C7 26.3 mm to (60.3, 43.8)
- moved 2C7A 26.3 mm to (63.5, 45.1)
- moved 2DA1 26.3 mm to (93.3, 37.8)
- moved 2R10 26.3 mm to (59.7, 37.1)
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Routing:
- net +IN: track 66.0 -> 57.0 mm
- net N$30: track 8.65 -> 1.11 mm
- net N$17: track 26.7 -> 29.6 mm
- net -IN: track 88.4 -> 89.9 mm
- net N$11: track 8.84 -> 7.62 mm
- net +16IN: track 25.8 -> 25.3 mm

Commit message: ..
Parts:
- added 3C1, 3C4: 100n, rcl:C0805
- added 3R1: 10k, rcl:R0805
- added 3R2: (no value), rcl:R0805
- added 3R3, 3R4, 3R5, 3R8: 270, rcl:R0805
- added U$1: (no value), SpeccyPower5v:_L
- 2VT1: value 2SK1984 -> IRF740
- 3R6: value 10k -> 270
- 3R7: value (none) -> 270
- moved 2R4 11.1 mm to (79.1, 33.0), turned to 0 degrees
- moved 2C2 9.25 mm to (51.8, 17.3), turned to 90 degrees
- moved 2VD1 9.23 mm to (78.7, 35.2), turned to 180 degrees
- moved 2VD2 6.54 mm to (59.5, 19.4), turned to 0 degrees
- moved 1VD1 5.72 mm to (44.5, 33.0), turned to 180 degrees
- moved 3R7 5.12 mm to (103.2, 27.6), turned to 270 degrees
- moved 3R6 5.12 mm to (105.4, 27.6), turned to 270 degrees
- moved 2VT1 2.88 mm to (59.7, 24.1)
- moved 1VD3 2.84 mm to (47.3, 29.8)
- moved 1VD4 1.31 mm to (47.0, 17.5), turned to 90 degrees
- moved 2R11 1.27 mm to (56.5, 36.2)
- moved 2R3 0.71 mm to (63.5, 15.2)
- moved T1 0.64 mm to (85.4, 21.9)
- moved 2VD3 0.45 mm to (66.0, 27.0)
- moved 2R16 0.45 mm to (94.3, 34.0)
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Connections:
- removed net N$24: 2VD1.A, T1.1
- new net N$6: 2R4.1, 2VD1.A
- net +16IN: now also 2VD1.C; no longer 2R4.1
- net +5V: now also 3C4.1, 3R1.2, 3R2.2, 3R3.1, 3R4.1, 3R5.1, 3R6.1, 3R7.1, 3R8.1; no longer 3R6.2, 3R7.2
- net GND: now also 3C1.2, 3C4.2, 3R3.2, 3R4.2, 3R5.2, 3R6.2, 3R7.2, 3R8.2
- net N$13: now also 3C1.1
- net N$22: now also T1.1; no longer 2VD1.C
- net N$26: now also 3R1.1, 3R2.1; no longer 3R6.1, 3R7.1
Routing:
- net +5V: track 25.9 -> 41.9 mm
- net GND: track 52.5 -> 67.8 mm
- net +IN: track 57.0 -> 66.6 mm
- net N$17: track 29.6 -> 22.4 mm
- net N$30: track 1.11 -> 7.25 mm
- net N$21: track 12.7 -> 9.00 mm
- net N$24: track 3.04 -> 0.00 mm
- net N$11: track 7.62 -> 4.76 mm
- net N$6: track 0.00 -> 2.26 mm
- net N$20: track 28.0 -> 26.2 mm
- net N$22: track 1.81 -> 3.34 mm
- net N$13: track 71.8 -> 70.4 mm
- net +16IN: track 25.3 -> 26.5 mm
- net N$44: track 9.19 -> 10.2 mm
- net N$37: track 6.10 -> 5.41 mm
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- added copper zone on layer 16, net N$23
Other:
- board text added: "220V"

Commit message: ..
Changed lines of the file:
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@@
 <wire x1="6.6675" y1="10.4775" x2="118.745" y2="10.4775" width="0.254" layer="20"/>
 <dimension x1="120.9675" y1="47.3075" x2="121.285" y2="10.4775" x3="125.095" y3="28.8925" layer="21" dtype="vertical"/>
-<text x="115.57" y="31.115" size="1.778" layer="16" font="vector" ratio="15" rot="MR90">5V 3A</text>
+<text x="116.205" y="30.48" size="1.778" layer="16" font="vector" ratio="15" rot="MR90.1">5V 3A</text>
 <wire x1="118.745" y1="47.3075" x2="6.6675" y2="47.3075" width="0.254" layer="20"/>
 <wire x1="118.745" y1="10.4775" x2="118.745" y2="47.3075" width="0.254" layer="20"/>
-<text x="33.655" y="21.2725" size="1.778" layer="16" font="vector" ratio="15" rot="MR90">github.com/74ls00</text>
+<text x="33.655" y="21.2725" size="1.778" layer="16" font="vector" ratio="15" rot="MR90.1">github.com/74ls00</text>
 <wire x1="75.565" y1="34.6075" x2="73.66" y2="36.5125" width="0.4064" layer="255"/>
 <wire x1="73.66" y1="36.5125" x2="67.6275" y2="36.5125" width="0.4064" layer="255"/>
 <wire x1="67.6275" y1="36.5125" x2="57.785" y2="46.0375" width="0.4064" layer="255"/>
 <wire x1="57.785" y1="46.0375" x2="50.8" y2="45.4025" width="0.4064" layer="255"/>
-<text x="8.89" y="26.035" size="1.778" layer="16" font="vector" ratio="15" rot="MR90">220V</text>
+<text x="8.89" y="26.035" size="1.778" layer="16" font="vector" ratio="15" rot="MR90.1">220V</text>
 </plain>
 <attributes>
