File: SpeccyPower5v.brd (EAGLE design)
At the start: 112.1 x 36.8 mm, 71 parts, among them T1 TRANS_ER29

Commit message: ..
Parts:
- 1R1, 1R2, 1R3, 1R4: value 470k -> 170k
- 3R8: value 270 -> (none)
- 3VD2: value (none) -> DTV32F
- turned 2VD4 to 175 degrees
Routing:
- net GND: track 67.8 -> 74.4 mm
- net +5V: track 41.9 -> 38.4 mm
- net N$13: track 70.4 -> 71.0 mm

Commit message: ..
Parts:
- 1C7: value 47x400v -> 22x400v
- renumbered 3L2 to 3L1
Changed lines of the file:
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@@
 <attribute name="VALUE" x="91.1225" y="30.7975" size="1.27" layer="28" rot="MR180"/>
 </element>
-<element name="1C7" library="SpeccyPower5v" package="TT5D11L" value="47x400v" x="53.6575" y="40.64" smashed="yes" rot="R90">
+<element name="1C7" library="SpeccyPower5v" package="TT5D11L" value="22x400v" x="53.6575" y="40.64" smashed="yes" rot="R90">
 <attribute name="NAME" x="32.9875" y="44.9185" size="1.27" layer="25" ratio="10"/>
 <attribute name="VALUE" x="39.275" y="44.363" size="1.27" layer="27" ratio="10" rot="R180"/>
@@
 <attribute name="VALUE" x="103.212896875" y="29.997396875" size="1.27" layer="27" ratio="10"/>
 </element>
-<element name="3L2" library="rcl" package="LAL02" value="mhn" x="104.14" y="43.815" smashed="yes" rot="R225">
+<element name="3L1" library="rcl" package="LAL02" value="mhn" x="104.14" y="43.815" smashed="yes" rot="R225">
 <attribute name="NAME" x="102.901853125" y="46.153575" size="0.9906" layer="25" ratio="10" rot="R225"/>
 <attribute name="VALUE" x="105.8346875" y="45.4631125" size="0.9906" layer="27" ratio="10" rot="R225"/>
@@
 </element>
 <element name="T1" library="SpeccyPower5v" package="ER29" value="TRANS_ER29" x="85.4075" y="21.9075" smashed="yes">
-<attribute name="NAME" x="84.59" y="23.955" size="1.27" layer="25"/>
+<attribute name="NAME" x="84.9075" y="29.3525" size="1.27" layer="25"/>
 </element>
 <element name="2R1A" library="rcl" package="M0805" value="120k" x="50.4825" y="39.37" smashed="yes" rot="MR180">
@@
 <contactref element="2R12" pad="2"/>
 <contactref element="3C2" pad="+"/>
-<contactref element="3L2" pad="1"/>
+<contactref element="3L1" pad="1"/>
 <wire x1="91.7575" y1="41.91" x2="91.7575" y2="41.9125" width="1.016" layer="16"/>
 <contactref element="3VD2" pad="C"/>
@@
 </signal>
 <signal name="+5V">
-<contactref element="3L2" pad="2"/>
+<contactref element="3L1" pad="2"/>
 <contactref element="3C3" pad="+"/>
 <contactref element="3R1" pad="2"/>
