File: SpeccyPower5v.sch (EAGLE design)
At the start: 67 parts, among them T1 TRANS_ER29

Commit message: .
Parts:
- removed 1RZ1: S1210, varistor:S1210
- removed 2R1: 220k 1w, rcl:R-EU_0613/15
- removed 2R1A1, 2R1C1, 2R1E1: 120k, rcl:R-EU_M0805
- removed 2R1B1, 2R1D1, 2R1F1: 150k, rcl:R-EU_M0805
- removed 3R1, 3R2: 0, rcl:R-EU_M1206
- added 3R8: (no value), rcl:R-EU_R0805
- added S1, S2: (no value), pinhead:PINHD-1X1
- 3VD2: value MA10799 -> (none); device diode:BYV32 -> diode:DIODE-DO220S
Connections:
- removed net N$27: 2R1C1.1, 2R1D1.1, 2R1E1.2, 2R1F1.1
- removed net N$31: 2R1A1.1, 2R1B1.1, 2R1C1.2, 2R1D1.2
- removed net N$33: 2C11.1, 3R2.1
- new net N$36: S2.1, SV1.1
- net +5V: now also 3R8.2
- net -IN: now also 2C11.1; no longer 3R2.2
- net N$26: now also 3R8.1
- net N$28: now also 3VD2.A; no longer 3VD2.A1, 3VD2.A2
- net N$32: now also S1.1; no longer SV1.1
Other:
- moved on the sheet: 1C2, 1F1, 1L1, 1PC1, 1R1, 1R2, 1R3, 1R4, 1TH1, 2C10, 2C11, 2C2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

Commit message: test v h
Parts:
- added 2C4A, 2C5A, 2C7A: (no value), rcl:C-EUC0805
Connections:
- net N$23 renamed +IN
- removed net N$40: 1DA1.VFB, 1PC1.EMIT, 2C4.2, 2R5.1, 2R7.2
- removed net N$6: 1DA1.COMP, 2C4.1, 2R5.2
- new net 817-3: 1DA1.VFB, 1PC1.EMIT, 2C4.2, 2C4A.2, 2R5.1, 2R7.2
- new net COMP: 1DA1.COMP, 2C4.1, 2C4A.1, 2R5.2
- net -IN: now also 2C5A.2, 2C7A.2
- net N$3: now also 2C5A.1
- net N$4: now also 2C7A.1
Other:
- moved on the sheet: 1C2, 1C7, 1F1, 1L1, 1R1, 1R2, 1R3, 1R4, 1TH1, 1VD1, 1VD2, 1VD3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

Commit message: ..
Parts:
- 2R13: device rcl:R-EU_0207/10 -> rcl:R-EU_0204/7
- 2VD2: device SpeccyPower5v:1N4148DO35-10 -> SpeccyPower5v:1N4148DO35-7
- 3L2: device rcl:L-USTFI0305 -> rcl:L-USLAL02
- 3R7: device rcl:R-EU_M1206 -> rcl:R-EU_M0805
Changed lines of the file:
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@@
 <part name="2VD3" library="SpeccyPower5v" deviceset="1N4148" device="DO35-7" value="1N4148"/>
 <part name="2R12" library="rcl" deviceset="R-EU_" device="R0805" value="910"/>
-<part name="2R13" library="rcl" deviceset="R-EU_" device="0207/10" value="820"/>
+<part name="2R13" library="rcl" deviceset="R-EU_" device="0204/7" value="820"/>
 <part name="2DA1" library="v-reg" deviceset="TL431CLP" device="" value="TL431"/>
 <part name="2R14" library="rcl" deviceset="R-EU_" device="R0805" value="47k*"/>
@@
 <part name="1F1" library="fuse" deviceset="SHK20L" device=""/>
 <part name="GND5" library="supply1" deviceset="GND" device=""/>
-<part name="2VD2" library="SpeccyPower5v" deviceset="1N4148" device="DO35-10" value="FR207"/>
+<part name="2VD2" library="SpeccyPower5v" deviceset="1N4148" device="DO35-7" value="FR207"/>
 <part name="1VD1" library="diode" deviceset="1N4004" device="" value="1N4007"/>
 <part name="1VD2" library="diode" deviceset="1N4004" device="" value="1N4007"/>
@@
 <part name="3C2" library="SpeccyPower5v" deviceset="CPOL-EU" device="TT2D7L" value="2200mfx10v"/>
 <part name="3C3" library="SpeccyPower5v" deviceset="CPOL-EU" device="TT2D7L" value="3300mfx6.3v"/>
-<part name="3L2" library="rcl" deviceset="L-US" device="TFI0305" value="mhn"/>
+<part name="3L2" library="rcl" deviceset="L-US" device="LAL02" value="mhn"/>
 <part name="GND9" library="supply1" deviceset="GND" device=""/>
 <part name="GND10" library="supply1" deviceset="GND" device=""/>
@@
 <part name="SV2" library="con-lstb" deviceset="MA03-1" device="" value="+5v"/>
 <part name="GND1" library="supply1" deviceset="GND" device=""/>
-<part name="3R7" library="rcl" deviceset="R-EU_" device="M1206" value="0"/>
+<part name="3R7" library="rcl" deviceset="R-EU_" device="M0805" value="0"/>
 <part name="3VD2" library="diode" deviceset="DIODE-" device="DO220S"/>
 <part name="3R8" library="rcl" deviceset="R-EU_" device="R0805"/>

Commit message: ..
Other:
- moved on the sheet: SV1

Commit message: ..
Parts:
- removed 3R8: (no value), rcl:R-EU_R0805
- 3C3: device SpeccyPower5v:CPOL-EUTT2D7L -> SpeccyPower5v:CPOL-EUTT2D7L-2
- 3R7: value 0 -> (none); device rcl:R-EU_M0805 -> rcl:R-EU_R0805
Connections:
- removed net N$42: 2C10.1, 2DA1.R, 2R16.2, 3R7.1
- net +5V: now also 3R7.2; no longer 3R8.2
- net N$26: now also 2C10.1, 2DA1.R, 2R16.2, 3R7.1; no longer 3R7.2, 3R8.1
Other:
- moved on the sheet: 3R7

Commit message: ..
Parts:
- 2R9: device rcl:R-EU_0207/10 -> rcl:R-EU_0204/7
- 2VD2: device SpeccyPower5v:1N4148DO35-7 -> SpeccyPower5v:1N4148DO35-10
Changed lines of the file:
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@@
 <part name="2R5" library="rcl" deviceset="R-EU_" device="0207/10" value="10k"/>
 <part name="2C3" library="rcl" deviceset="CPOL-EU" device="E2.5-6" value="100x25v"/>
-<part name="2R9" library="rcl" deviceset="R-EU_" device="0207/10" value="100"/>
+<part name="2R9" library="rcl" deviceset="R-EU_" device="0204/7" value="100"/>
 <part name="2VD3" library="SpeccyPower5v" deviceset="1N4148" device="DO35-7" value="1N4148"/>
 <part name="2R12" library="rcl" deviceset="R-EU_" device="R0805" value="910"/>
@@
 <part name="1F1" library="fuse" deviceset="SHK20L" device=""/>
 <part name="GND5" library="supply1" deviceset="GND" device=""/>
-<part name="2VD2" library="SpeccyPower5v" deviceset="1N4148" device="DO35-7" value="FR207"/>
+<part name="2VD2" library="SpeccyPower5v" deviceset="1N4148" device="DO35-10" value="FR207"/>
 <part name="1VD1" library="diode" deviceset="1N4004" device="" value="1N4007"/>
 <part name="1VD2" library="diode" deviceset="1N4004" device="" value="1N4007"/>

Commit message: ..
Parts:
- added 3C1, 3C4: 100n, rcl:C-EUC0805
- added 3R1: 10k, rcl:R-EU_R0805
- added 3R2: (no value), rcl:R-EU_R0805
- added 3R3, 3R4, 3R5, 3R8: 270, rcl:R-EU_R0805
- 2VT1: value 2SK1984 -> IRF740
- 3R6: value 10k -> 270
- 3R7: value (none) -> 270
Connections:
- removed net N$24: 2VD1.A, T1.OP1
- new net N$6: 2R4.1, 2VD1.A
- net +16IN: now also 2VD1.C; no longer 2R4.1
- net +5V: now also 3C4.1, 3R1.2, 3R2.2, 3R3.1, 3R4.1, 3R5.1, 3R6.1, 3R7.1, 3R8.1; no longer 3R6.2, 3R7.2
- net GND: now also 3C1.2, 3C4.2, 3R3.2, 3R4.2, 3R5.2, 3R6.2, 3R7.2, 3R8.2
- net N$13: now also 3C1.1
- net N$22: now also T1.OP1; no longer 2VD1.C
- net N$26: now also 3R1.1, 3R2.1; no longer 3R6.1, 3R7.1
Other:
- note added: "5V 3A"
- note added: "github.com/74ls00/SpeccyPower5v"
- note removed: "github.com/74ls00"
- moved on the sheet: 1C2, 1C7, 1DA1, 1F1, 1L1, 1PC1, 1R1, 1R2, 1R3, 1R4, 1TH1, 1VD1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

Commit message: ..
Other:
- note added: "T1 ETD 22/16/9 0.3mm I 4-5 81w 0.25mm II 1-3 12w 0.2mm III 6-9 7w x7 0.55mm"
- note removed: "2T1 ETD 29/16/10 2mm I 2-4 51w 0.4mm II 4-5 51w 0.4mm III 1-3 17w 0.2mm IV 6-7 5w 6x0.55mm V 10-11 8w 4x0.55mm"
Changed lines of the file:
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@@
 <plain>
 <text x="284.48" y="10.16" size="3.81" layer="91" rot="R180">github.com/74ls00/SpeccyPower5v</text>
-<text x="200.66" y="43.18" size="0.1778" layer="91" font="vector" rot="MR180">2T1 ETD 29/16/10 2mm
-I   2-4 51w 0.4mm
-II 4-5 51w 0.4mm
-III  1-3 17w 0.2mm
-IV 6-7 5w 6x0.55mm
-V 10-11 8w 4x0.55mm</text>
+<text x="200.66" y="43.18" size="1.778" layer="91" font="vector" rot="MR180">T1 ETD 22/16/9 0.3mm
+I    4-5 81w 0.25mm
+II   1-3 12w 0.2mm
+III  6-9 7w x7 0.55mm
+</text>
 <wire x1="167.64" y1="116.84" x2="167.64" y2="0" width="0.3048" layer="98" style="shortdash"/>
 <wire x1="292.1" y1="116.84" x2="167.64" y2="116.84" width="0.4064" layer="98" style="shortdash"/>
