File: SpeccyPower5v.sch (EAGLE design)
At the start: 70 parts, among them T1 TRANS_ER29

Commit message: ..
Parts:
- 1R1, 1R2, 1R3, 1R4: value 470k -> 170k
- 3R8: value 270 -> (none)
- 3VD2: value (none) -> DTV32F
Other:
- moved on the sheet: 1F1, 3R3, 3R4, 3R5, 3R6, 3R7, 3R8, S1, S2, SV1, SV2

Commit message: ..
Parts:
- 1C7: value 47x400v -> 22x400v
- renumbered 3L2 to 3L1
Other:
- note added: "T1 ETD 22/16/9 0.3mm (ZEBRA 4TP PM-EEH22A-25) I 4-5 43+43w 0.2mm II 1-3 13w 0.2mm III 6-9 4w x4 0.56mm"
- note removed: "T1 ETD 22/16/9 0.3mm I 4-5 81w 0.25mm II 1-3 12w 0.2mm III 6-9 7w x7 0.55mm"
Changed lines of the file:
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@@
 <part name="GND2" library="supply1" deviceset="GND" device=""/>
 <part name="GND3" library="supply1" deviceset="GND" device=""/>
-<part name="1C7" library="SpeccyPower5v" deviceset="CPOL-EU" device="TT5D11L" value="47x400v"/>
+<part name="1C7" library="SpeccyPower5v" deviceset="CPOL-EU" device="TT5D11L" value="22x400v"/>
 <part name="2VT1" library="transistor-power" deviceset="IRF3704" device="L-V" value="IRF740"/>
 <part name="2R10" library="rcl" deviceset="R-EU_" device="0207/10" value="470"/>
@@
 <part name="3C2" library="SpeccyPower5v" deviceset="CPOL-EU" device="TT2D7L" value="2200mfx10v"/>
 <part name="3C3" library="SpeccyPower5v" deviceset="CPOL-EU" device="TT2D7L-2" value="3300mfx6.3v"/>
-<part name="3L2" library="rcl" deviceset="L-US" device="LAL02" value="mhn"/>
+<part name="3L1" library="rcl" deviceset="L-US" device="LAL02" value="mhn"/>
 <part name="GND9" library="supply1" deviceset="GND" device=""/>
 <part name="GND10" library="supply1" deviceset="GND" device=""/>
@@
 <plain>
 <text x="266.7" y="10.16" size="3.81" layer="98" rot="R180">github.com/74ls00/SpeccyPower5v</text>
-<text x="203.2" y="43.18" size="1.778" layer="98" font="vector" rot="MR180">T1 ETD 22/16/9 0.3mm
-I    4-5 81w 0.25mm
-II   1-3 12w 0.2mm
-III  6-9 7w x7 0.55mm
+<text x="198.12" y="43.18" size="1.778" layer="98" font="vector" rot="MR180">T1 ETD 22/16/9 0.3mm
+(ZEBRA 4TP PM-EEH22A-25)
+I    4-5 43+43w 0.2mm
+II   1-3   13w  0.2mm
+III  6-9  4w x4  0.56mm
 </text>
 <wire x1="167.64" y1="116.84" x2="167.64" y2="0" width="0.3048" layer="98" style="shortdash"/>
@@
 <attribute name="VALUE" x="237.363" y="109.7026" size="1.778" layer="96"/>
 </instance>
-<instance part="3L2" gate="G$1" x="223.52" y="106.68" smashed="yes" rot="R90">
+<instance part="3L1" gate="G$1" x="223.52" y="106.68" smashed="yes" rot="R90">
 <attribute name="NAME" x="218.44" y="111.76" size="1.778" layer="95"/>
 <attribute name="VALUE" x="223.52" y="109.22" size="1.778" layer="96"/>
@@
 <attribute name="VALUE" x="25.4" y="77.47" size="1.778" layer="96" rot="MR180"/>
 </instance>
-<instance part="1R1" gate="G$1" x="25.4" y="78.74" rot="MR180"/>
+<instance part="1R1" gate="G$1" x="25.4" y="78.74" smashed="yes" rot="MR180">
+<attribute name="NAME" x="21.59" y="82.3214" size="1.778" layer="95" rot="MR180"/>
+<attribute name="VALUE" x="21.59" y="76.962" size="1.778" layer="96" rot="MR180"/>
+</instance>
 <instance part="2R11" gate="G$1" x="139.7" y="53.34" smashed="yes" rot="R90">
 <attribute name="NAME" x="135.89" y="56.9214" size="1.778" layer="95" rot="R180"/>
@@
 <attribute name="NAME" x="41.91" y="99.822" size="1.778" layer="95"/>
 </instance>
-<instance part="1R2" gate="G$1" x="25.4" y="86.36" rot="MR180"/>
-<instance part="1R3" gate="G$1" x="25.4" y="101.6" rot="MR180"/>
-<instance part="1R4" gate="G$1" x="25.4" y="93.98" rot="MR180"/>
+<instance part="1R2" gate="G$1" x="25.4" y="86.36" smashed="yes" rot="MR180">
+<attribute name="NAME" x="21.59" y="89.9414" size="1.778" layer="95" rot="MR180"/>
+<attribute name="VALUE" x="21.59" y="84.582" size="1.778" layer="96" rot="MR180"/>
+</instance>
+<instance part="1R3" gate="G$1" x="25.4" y="101.6" smashed="yes" rot="MR180">
+<attribute name="NAME" x="21.59" y="105.1814" size="1.778" layer="95" rot="MR180"/>
+<attribute name="VALUE" x="21.59" y="99.822" size="1.778" layer="96" rot="MR180"/>
+</instance>
+<instance part="1R4" gate="G$1" x="25.4" y="93.98" smashed="yes" rot="MR180">
+<attribute name="NAME" x="21.59" y="97.5614" size="1.778" layer="95" rot="MR180"/>
+<attribute name="VALUE" x="21.59" y="92.202" size="1.778" layer="96" rot="MR180"/>
+</instance>
 <instance part="T1" gate="G$1" x="167.64" y="88.9" smashed="yes">
 <attribute name="NAME" x="162.56" y="109.22" size="1.27" layer="95"/>
@@
 <wire x1="203.2" y1="106.68" x2="213.36" y2="106.68" width="0.1524" layer="91"/>
 <wire x1="213.36" y1="106.68" x2="213.36" y2="104.14" width="0.1524" layer="91"/>
-<pinref part="3L2" gate="G$1" pin="1"/>
+<pinref part="3L1" gate="G$1" pin="1"/>
 <wire x1="215.9" y1="106.68" x2="213.36" y2="106.68" width="0.1524" layer="91"/>
 <junction x="213.36" y="106.68"/>
@@
 <net name="+5V" class="0">
 <segment>
-<pinref part="3L2" gate="G$1" pin="2"/>
+<pinref part="3L1" gate="G$1" pin="2"/>
 <pinref part="3C3" gate="G$1" pin="+"/>
 <wire x1="231.14" y1="106.68" x2="233.68" y2="106.68" width="0.1524" layer="91"/>
